File: 3003/3003.kicad_pcb (KiCad board)
At the start: 2 copper layers, 266 x 85 mm, 52 parts, among them SW1 1, SW10 5, SW11 6, SW12 A, SW13 BOOST, SW14 CE, SW15 SCALE, SW16 ←, SW17 7, SW18 8, SW19 9, SW2 2, SW20 µ, SW21 PREV MENU, SW22 SOFT 1, SW23 RESET, SW24 →, SW25 OPR STBY, SW26 EX SENSE, SW27 EX GRD, SW28 W BAND, SW29 NEW REF, SW3 K, SW30 OFFSET, SW31 LIMIT, SW32 SOFT 4, SW33 +1, SW34 0, SW35 M, SW36 m, SW37 dbm, SW38 SOFT 2, SW39 SOFT 3, SW4 Ω, SW40 SOFT 5, SW41 ., SW42 3, SW43 ENTER, SW44 V, SW45 x10, SW5 Hz, SW6 SPEC, SW7 ÷10, SW8 AMPL FREQ, SW9 4

Commit message: added more clearance around screw holes
Routing:
- net /ROW5: track 375.2 -> 384.0 mm
- net /COL6: track 164.6 -> 170.4 mm
- net /COL7: track 136.0 -> 140.5 mm
- net /COL5: track 134.8 -> 137.2 mm
- net /ROW3: track 309.6 -> 311.2 mm
- net /LED2B: track 105.8 -> 106.5 mm
